File: whitterm-hat/micro.sch (KiCad schematic (older format))
At the start: 25 parts, among them IC1 SAMD21G18A, J5 Conn_02x05_Odd_Even, Y1 32.768

Commit message: pcb sent for production
Parts:
- added R66: 110R, KiCad/Resistor_SMD.pretty:R_0603_1608Metric, symbol Device:R
- added SW2: SW_Push, mcous/kicad-lib/footprints/switch.pretty:SPST-4-PIN_6mm_sm, symbol Switch:SW_Push
- D8: footprint KiCad/Package_TO_SOT_THT.pretty:TO-92_Inline -> KiCad/Package_SO.pretty:SOIC-8_3.9x4.9mm_P1.27mm; symbol Reference_Voltage:LM285Z-1.2 -> Reference_Voltage:LM285D-1.2
- TP22, TP23, TP24: footprint KiCad/TestPoint.pretty:TestPoint_Pad_D2.0mm -> KiCad/TestPoint.pretty:TestPoint_Pad_D1.5mm
Connections:
- net labels added: RXD, TXD
- net labels removed: SAMD_RXD, SAMD_TXD
- wire segments 129 -> 134
Changed lines of the file:
@@
 EESchema Schematic File Version 4
 LIBS:whitterm-hat-cache
-EELAYER 26 0
+EELAYER 29 0
 EELAYER END
 $Descr A3 16535 11693
@@
 $EndComp
 $Comp
-L whitterm-hat-rescue:SAMD21G18A-jbr-ics IC1
+L whitterm-hat-rescue:SAMD21G18A-jbr-ics IC?
 U 1 1 5C61ABF0
 P 8050 4400
-AR Path="/5C61ABF0" Ref="IC1"  Part="1"
+AR Path="/5C61ABF0" Ref="IC?"  Part="1"
 AR Path="/5C619272/5C61ABF0" Ref="IC1"  Part="1"
 F 0 "IC1" H 8100 6369 100 0000 C CNN
@@
 Text HLabel 9900 5000 2    50   BiDi ~ 0
 SDA
-$Comp
-L Reference_Voltage:LM285Z-1.2 D8
-U 1 1 5C6D852D
-P 4300 3700
-F 0 "D8" V 4346 3612 50  0000 R CNN
-F 1 "LM285Z-1.2" V 4255 3612 50  0000 R CNN
-F 2 "KiCad/Package_TO_SOT_THT.pretty:TO-92_Inline" H 4300 3500 50  0001 C CIN
-F 3 "http://www.onsemi.com/pub_link/Collateral/LM285-D.PDF" H 4300 3700 50  0001 C CIN
-	1    4300 3700
-	0    -1   -1   0
-$EndComp
 $Comp
 L Device:R_Small R24
@@
 Wire Wire Line
 	13500 4250 13700 4250
-$Comp
-L power:VCC #PWR0130
-U 1 1 5C70C9A5
-P 14600 3600
-F 0 "#PWR0130" H 14600 3450 50  0001 C CNN
-F 1 "VCC" H 14617 3773 50  0000 C CNN
-F 2 "" H 14600 3600 50  0001 C CNN
-F 3 "" H 14600 3600 50  0001 C CNN
-	1    14600 3600
-	1    0    0    -1
-$EndComp
 Wire Wire Line
 	14600 3600 14600 3800
@@
 D-
 Text HLabel 5800 4700 0    60   Output ~ 0
-SAMD_TXD
+TXD
 Text HLabel 5800 4800 0    60   Input ~ 0
-SAMD_RXD
+RXD
 Text Label 10000 3900 0    60   ~ 0
 NRST
@@
 Text HLabel 9900 5400 2    60   Input ~ 0
 D10
-Text HLabel 9900 5600 2    60   Input ~ 0
-D11
 Text HLabel 6300 5300 0    60   Input ~ 0
 MISO
@@
 Wire Wire Line
 	9850 5400 9900 5400
-Wire Wire Line
-	9850 5600 9900 5600
 $Comp
 L Connector:TestPoint TP?
@@
 F 0 "TP23" H 5800 4900 50  0000 L CNN
 F 1 "TestPoint" H 5908 4729 50  0001 L CNN
-F 2 "KiCad/TestPoint.pretty:TestPoint_Pad_D2.0mm" H 6050 4700 50  0001 C CNN
+F 2 "KiCad/TestPoint.pretty:TestPoint_Pad_D1.5mm" H 6050 4700 50  0001 C CNN
 F 3 "~" H 6050 4700 50  0001 C CNN
 	1    5850 4700
@@
 F 0 "TP24" H 5950 5000 50  0000 L CNN
 F 1 "TestPoint" H 6008 4829 50  0001 L CNN
-F 2 "KiCad/TestPoint.pretty:TestPoint_Pad_D2.0mm" H 6150 4800 50  0001 C CNN
+F 2 "KiCad/TestPoint.pretty:TestPoint_Pad_D1.5mm" H 6150 4800 50  0001 C CNN
 F 3 "~" H 6150 4800 50  0001 C CNN
 	1    5950 4800
@@
 F 0 "TP22" H 4600 3600 50  0000 L CNN
 F 1 "TestPoint" H 4708 3429 50  0001 L CNN
-F 2 "KiCad/TestPoint.pretty:TestPoint_Pad_D2.0mm" H 4850 3400 50  0001 C CNN
+F 2 "KiCad/TestPoint.pretty:TestPoint_Pad_D1.5mm" H 4850 3400 50  0001 C CNN
 F 3 "~" H 4850 3400 50  0001 C CNN
 	1    4650 3400
@@
 Wire Wire Line
 	4650 3400 6350 3400
+$Comp
+L Reference_Voltage:LM285D-1.2 D8
+U 1 1 5C6D852D
+P 4300 3700
+F 0 "D8" V 4346 3612 50  0000 R CNN
+F 1 "LM285Z-1.2" V 4255 3612 50  0000 R CNN
+F 2 "KiCad/Package_SO.pretty:SOIC-8_3.9x4.9mm_P1.27mm" H 4300 3500 50  0001 C CIN
+F 3 "http://www.onsemi.com/pub_link/Collateral/LM285-D.PDF" H 4300 3700 50  0001 C CIN
+	1    4300 3700
+	0    -1   -1   0
+$EndComp
+$Comp
+L Switch:SW_Push SW2
+U 1 1 5CA712A5
+P 13550 7600
+F 0 "SW2" V 13596 7552 50  0000 R CNN
+F 1 "SW_Push" V 13505 7552 50  0000 R CNN
+F 2 "mcous/kicad-lib/footprints/switch.pretty:SPST-4-PIN_6mm_sm" H 13550 7800 50  0001 C CNN
+F 3 "~" H 13550 7800 50  0001 C CNN
+F 4 "TE" H 13550 7600 50  0001 C CNN "MFN"
+F 5 "4-1437565-1" H 13550 7600 50  0001 C CNN "MFP"
+	1    13550 7600
+	0    -1   -1   0
+$EndComp
+$Comp
+L Device:R R66
+U 1 1 5CA7190D
+P 13550 7050
+F 0 "R66" V 13343 7050 50  0000 C CNN
+F 1 "110R" V 13434 7050 50  0000 C CNN
+F 2 "KiCad/Resistor_SMD.pretty:R_0603_1608Metric" V 13480 7050 50  0001 C CNN
+F 3 "~" H 13550 7050 50  0001 C CNN
+	1    13550 7050
+	-1   0    0    -1
+$EndComp
+$Comp
+L power:GND #PWR024
+U 1 1 5CA72F91
+P 13550 7900
+F 0 "#PWR024" H 13550 7650 50  0001 C CNN
+F 1 "GND" H 13555 7727 50  0000 C CNN
+F 2 "" H 13550 7900 50  0001 C CNN
+F 3 "" H 13550 7900 50  0001 C CNN
+	1    13550 7900
+	1    0    0    -1
+$EndComp
+Wire Wire Line
+	13550 7800 13550 7900
+$Comp
+L power:VCC #PWR0130
+U 1 1 5C70C9A5
+P 14600 3600
+F 0 "#PWR0130" H 14600 3450 50  0001 C CNN
+F 1 "VCC" H 14617 3773 50  0000 C CNN
+F 2 "" H 14600 3600 50  0001 C CNN
+F 3 "" H 14600 3600 50  0001 C CNN
+	1    14600 3600
+	1    0    0    -1
+$EndComp
+$Comp
+L power:VCC #PWR023
+U 1 1 5CA82980
+P 13550 6750
+F 0 "#PWR023" H 13550 6600 50  0001 C CNN
+F 1 "VCC" H 13567 6923 50  0000 C CNN
+F 2 "" H 13550 6750 50  0001 C CNN
+F 3 "" H 13550 6750 50  0001 C CNN
+	1    13550 6750
+	1    0    0    -1
+$EndComp
+Wire Wire Line
+	13550 6900 13550 6750
+Wire Wire Line
+	13550 7200 13550 7300
+Wire Wire Line
+	13550 7300 13400 7300
+Connection ~ 13550 7300
+Wire Wire Line
+	13550 7300 13550 7400
+Wire Wire Line
+	9850 5600 10000 5600
+Text Label 10000 5600 0    50   ~ 0
+D11
+Text Label 13400 7300 2    50   ~ 0
+D11
 $EndSCHEMATC

Commit message: firmware added and bring up R value changes
Parts:
- R66: value 110R -> 10k
Changed lines of the file:
@@
 P 13550 7050
 F 0 "R66" V 13343 7050 50  0000 C CNN
-F 1 "110R" V 13434 7050 50  0000 C CNN
+F 1 "10k" V 13434 7050 50  0000 C CNN
 F 2 "KiCad/Resistor_SMD.pretty:R_0603_1608Metric" V 13480 7050 50  0001 C CNN
 F 3 "~" H 13550 7050 50  0001 C CNN

Commit message: mods during bring up, see notes
Parts:
- D8: value LM285Z-1.2 -> LM285D-2.5G; MFN (none) -> ON Semiconductor; MFP (none) -> LM285D-2.5GOS-ND
- R26, R27, R28: value 110R -> 150R
- Y1: MFN Micro Crystal -> Abracon LLC; MFP CM8V-32.768-TA-020-7 -> ABS06-127-32.768KHZ-T
Changed lines of the file:
@@
 F 2 "StefanHamminga/SH_Crystals_Oscillators.pretty:Crystal_2-SMD_2x1.2mm" H 5700 2500 50  0001 C CNN
 F 3 "https://docs-emea.rs-online.com/webdocs/0f59/0900766b80f59f41.pdf" H 5700 2500 50  0001 C CNN
-F 4 " Micro Crystal" H 5700 2500 60  0001 C CNN "MFN"
-F 5 "CM8V-32.768-TA-020-7 " H 5700 2500 60  0001 C CNN "MFP"
+F 4 "Abracon LLC" H 5700 2500 60  0001 C CNN "MFN"
+F 5 "ABS06-127-32.768KHZ-T	" H 5700 2500 60  0001 C CNN "MFP"
 	1    5700 2500
 	1    0    0    -1
@@
 P 13350 3800
 F 0 "R26" V 13143 3800 50  0000 C CNN
-F 1 "110R" V 13234 3800 50  0000 C CNN
+F 1 "150R" V 13234 3800 50  0000 C CNN
 F 2 "KiCad/Resistor_SMD.pretty:R_0603_1608Metric" V 13280 3800 50  0001 C CNN
 F 3 "~" H 13350 3800 50  0001 C CNN
@@
 P 13350 4250
 F 0 "R27" V 13143 4250 50  0000 C CNN
-F 1 "110R" V 13234 4250 50  0000 C CNN
+F 1 "150R" V 13234 4250 50  0000 C CNN
 F 2 "KiCad/Resistor_SMD.pretty:R_0603_1608Metric" V 13280 4250 50  0001 C CNN
 F 3 "~" H 13350 4250 50  0001 C CNN
@@
 P 13350 4700
 F 0 "R28" V 13143 4700 50  0000 C CNN
-F 1 "110R" V 13234 4700 50  0000 C CNN
+F 1 "150R" V 13234 4700 50  0000 C CNN
 F 2 "KiCad/Resistor_SMD.pretty:R_0603_1608Metric" V 13280 4700 50  0001 C CNN
 F 3 "~" H 13350 4700 50  0001 C CNN
@@
 P 4300 3700
 F 0 "D8" V 4346 3612 50  0000 R CNN
-F 1 "LM285Z-1.2" V 4255 3612 50  0000 R CNN
+F 1 "LM285D-2.5G" V 4255 3612 50  0000 R CNN
 F 2 "KiCad/Package_SO.pretty:SOIC-8_3.9x4.9mm_P1.27mm" H 4300 3500 50  0001 C CIN
 F 3 "http://www.onsemi.com/pub_link/Collateral/LM285-D.PDF" H 4300 3700 50  0001 C CIN
+F 4 "ON Semiconductor" H 4300 3700 50  0001 C CNN "MFN"
+F 5 "LM285D-2.5GOS-ND " H 4300 3700 50  0001 C CNN "MFP"
 	1    4300 3700
 	0    -1   -1   0
