File: whitterm-hat/buffers.sch (KiCad schematic (older format))
At the start: 50 parts, among them Q3 BC850, Q4 BC850, Q5 BC850, Q6 BC850, U10 ADA4807-2ARM, U11 ADA4807-2ARM

Commit message: pcb sent for production
Parts:
- removed TP28: TestPoint, KiCad/TestPoint.pretty:TestPoint_Pad_D2.0mm, symbol Connector:TestPoint
- TP29, TP30, TP31, TP32, TP33: footprint KiCad/TestPoint.pretty:TestPoint_Pad_D2.0mm -> KiCad/TestPoint.pretty:TestPoint_Pad_D1.5mm
Connections:
- wire segments 157 -> 156
Changed lines of the file:
@@
 EESchema Schematic File Version 4
 LIBS:whitterm-hat-cache
-EELAYER 26 0
+EELAYER 29 0
 EELAYER END
 $Descr A3 16535 11693
@@
 Text HLabel 1400 2700 0    50   Input ~ 0
 AIN_I1
-Wire Wire Line
-	1400 2700 1700 2700
 $Comp
 L Device:R R38
@@
 Wire Wire Line
 	5900 1850 5900 2000
-$Comp
-L Diode:BAV99 D17
-U 1 1 5C674D27
-P 3650 2150
-F 0 "D17" H 3650 1925 50  0000 C CNN
-F 1 "BAV99" H 3650 2016 50  0000 C CNN
-F 2 "KiCad/Package_TO_SOT_SMD.pretty:SOT-23" H 3650 2000 50  0001 C CNN
-F 3 "www.nxp.com/documents/data_sheet/BAV99_SER.pdf" H 3650 2250 50  0001 C CNN
-	1    3650 2150
-	-1   0    0    1
-$EndComp
-$Comp
-L Diode:BAV99 D16
-U 1 1 5C674E30
-P 3350 2150
-F 0 "D16" H 3350 1925 50  0000 C CNN
-F 1 "BAV99" H 3350 2016 50  0000 C CNN
-F 2 "KiCad/Package_TO_SOT_SMD.pretty:SOT-23" H 3350 2000 50  0001 C CNN
-F 3 "www.nxp.com/documents/data_sheet/BAV99_SER.pdf" H 3350 2250 50  0001 C CNN
-	1    3350 2150
-	-1   0    0    1
-$EndComp
 Wire Wire Line
 	3500 2150 3500 2700
-Connection ~ 3500 2150
 Wire Wire Line
 	3850 4900 3750 4900
@@
 Wire Wire Line
 	3550 4700 3850 4700
-$Comp
-L Diode:BAV99 D17
-U 2 1 5C6794A5
-P 3700 4150
-F 0 "D17" H 3700 3925 50  0000 C CNN
-F 1 "BAV99" H 3700 4016 50  0000 C CNN
-F 2 "KiCad/Package_TO_SOT_SMD.pretty:SOT-23" H 3700 4000 50  0001 C CNN
-F 3 "www.nxp.com/documents/data_sheet/BAV99_SER.pdf" H 3700 4250 50  0001 C CNN
-	2    3700 4150
-	-1   0    0    1
-$EndComp
-$Comp
-L Diode:BAV99 D16
-U 2 1 5C6794AC
-P 3400 4150
-F 0 "D16" H 3400 3925 50  0000 C CNN
-F 1 "BAV99" H 3400 4016 50  0000 C CNN
-F 2 "KiCad/Package_TO_SOT_SMD.pretty:SOT-23" H 3400 4000 50  0001 C CNN
-F 3 "www.nxp.com/documents/data_sheet/BAV99_SER.pdf" H 3400 4250 50  0001 C CNN
-	2    3400 4150
-	-1   0    0    1
-$EndComp
 Wire Wire Line
 	3550 4150 3550 4700
-Connection ~ 3550 4150
 Text Notes 2450 1500 0    50   ~ 0
 0-10 V input to 0-3 V for uC ADC. G = 3/10
@@
 $Comp
 L Connector:TestPoint TP?
-U 1 1 5D675C23
-P 1700 2700
-AR Path="/5D675C23" Ref="TP?"  Part="1"
-AR Path="/5C67462C/5D675C23" Ref="TP28"  Part="1"
-F 0 "TP28" H 1758 2774 50  0000 L CNN
-F 1 "TestPoint" H 1758 2729 50  0001 L CNN
-F 2 "KiCad/TestPoint.pretty:TestPoint_Pad_D2.0mm" H 1900 2700 50  0001 C CNN
-F 3 "~" H 1900 2700 50  0001 C CNN
-	1    1700 2700
-	1    0    0    -1
-$EndComp
-$Comp
-L Connector:TestPoint TP?
 U 1 1 5D67A81A
 P 4950 2800
@@
 F 0 "TP30" H 5008 2874 50  0000 L CNN
 F 1 "TestPoint" H 5008 2829 50  0001 L CNN
-F 2 "KiCad/TestPoint.pretty:TestPoint_Pad_D2.0mm" H 5150 2800 50  0001 C CNN
+F 2 "KiCad/TestPoint.pretty:TestPoint_Pad_D1.5mm" H 5150 2800 50  0001 C CNN
 F 3 "~" H 5150 2800 50  0001 C CNN
 	1    4950 2800
@@
 F 0 "TP29" H 2758 8874 50  0000 L CNN
 F 1 "TestPoint" H 2758 8829 50  0001 L CNN
-F 2 "KiCad/TestPoint.pretty:TestPoint_Pad_D2.0mm" H 2900 8800 50  0001 C CNN
+F 2 "KiCad/TestPoint.pretty:TestPoint_Pad_D1.5mm" H 2900 8800 50  0001 C CNN
 F 3 "~" H 2900 8800 50  0001 C CNN
 	1    2700 8800
@@
 F 0 "TP31" H 5408 8974 50  0000 L CNN
 F 1 "TestPoint" H 5408 8929 50  0001 L CNN
-F 2 "KiCad/TestPoint.pretty:TestPoint_Pad_D2.0mm" H 5550 8900 50  0001 C CNN
+F 2 "KiCad/TestPoint.pretty:TestPoint_Pad_D1.5mm" H 5550 8900 50  0001 C CNN
 F 3 "~" H 5550 8900 50  0001 C CNN
 	1    5350 8900
@@
 F 0 "TP32" H 8608 2274 50  0000 L CNN
 F 1 "TestPoint" H 8608 2229 50  0001 L CNN
-F 2 "KiCad/TestPoint.pretty:TestPoint_Pad_D2.0mm" H 8750 2200 50  0001 C CNN
+F 2 "KiCad/TestPoint.pretty:TestPoint_Pad_D1.5mm" H 8750 2200 50  0001 C CNN
 F 3 "~" H 8750 2200 50  0001 C CNN
 	1    8550 2200
@@
 F 0 "TP33" H 12808 1624 50  0000 L CNN
 F 1 "TestPoint" H 12808 1579 50  0001 L CNN
-F 2 "KiCad/TestPoint.pretty:TestPoint_Pad_D2.0mm" H 12950 1550 50  0001 C CNN
+F 2 "KiCad/TestPoint.pretty:TestPoint_Pad_D1.5mm" H 12950 1550 50  0001 C CNN
 F 3 "~" H 12950 1550 50  0001 C CNN
 	1    12750 1550
@@
 Wire Wire Line
 	4950 2800 5300 2800
-Connection ~ 1700 2700
-Wire Wire Line
-	1700 2700 2000 2700
 Wire Wire Line
 	2700 8800 2500 8800
@@
 Text Notes 3250 6750 0    50   ~ 0
 0-10 V output to 0-3.3 V for uC DAC. G = 3 ((100 / 50) + 1)
+$Comp
+L Diode:BAV99 D17
+U 1 1 5C914FDF
+P 3350 2150
+F 0 "D17" H 3350 1925 50  0000 C CNN
+F 1 "BAV99" H 3350 2016 50  0000 C CNN
+F 2 "KiCad/Package_TO_SOT_SMD.pretty:SOT-23" H 3350 2000 50  0001 C CNN
+F 3 "https://assets.nexperia.com/documents/data-sheet/BAV99_SER.pdf" H 3350 2250 50  0001 C CNN
+	1    3350 2150
+	-1   0    0    1
+$EndComp
+$Comp
+L Diode:BAV99 D16
+U 1 1 5C8F8B33
+P 3400 4150
+F 0 "D16" H 3400 3925 50  0000 C CNN
+F 1 "BAV99" H 3400 4016 50  0000 C CNN
+F 2 "KiCad/Package_TO_SOT_SMD.pretty:SOT-23" H 3400 4000 50  0001 C CNN
+F 3 "https://assets.nexperia.com/documents/data-sheet/BAV99_SER.pdf" H 3400 4250 50  0001 C CNN
+	1    3400 4150
+	-1   0    0    1
+$EndComp
+$Comp
+L Diode:BAV99 D17
+U 2 1 5C8F9AE0
+P 3650 2150
+F 0 "D17" H 3650 1925 50  0000 C CNN
+F 1 "BAV99" H 3650 2016 50  0000 C CNN
+F 2 "KiCad/Package_TO_SOT_SMD.pretty:SOT-23" H 3650 2000 50  0001 C CNN
+F 3 "https://assets.nexperia.com/documents/data-sheet/BAV99_SER.pdf" H 3650 2250 50  0001 C CNN
+	2    3650 2150
+	-1   0    0    1
+$EndComp
+Connection ~ 3500 2150
+$Comp
+L Diode:BAV99 D16
+U 2 1 5C93469F
+P 3700 4150
+F 0 "D16" H 3700 3925 50  0000 C CNN
+F 1 "BAV99" H 3700 4016 50  0000 C CNN
+F 2 "KiCad/Package_TO_SOT_SMD.pretty:SOT-23" H 3700 4000 50  0001 C CNN
+F 3 "https://assets.nexperia.com/documents/data-sheet/BAV99_SER.pdf" H 3700 4250 50  0001 C CNN
+	2    3700 4150
+	-1   0    0    1
+$EndComp
+Connection ~ 3550 4150
+Wire Wire Line
+	1400 2700 2000 2700
 $EndSCHEMATC

Commit message: button button logic
Parts:
- D14, D15: value BZX84Cxx -> BZX84C10LT1G
Changed lines of the file:
@@
 P 2000 3000
 F 0 "D14" V 1954 3079 50  0000 L CNN
-F 1 "BZX84Cxx" V 2045 3079 50  0000 L CNN
+F 1 "BZX84C10LT1G" V 2045 3079 50  0000 L CNN
 F 2 "KiCad/Diode_SMD.pretty:D_SOT-23_ANK" H 2000 2825 50  0001 C CNN
 F 3 "https://diotec.com/tl_files/diotec/files/pdf/datasheets/bzx84c2v4.pdf" H 2000 3000 50  0001 C CNN
@@
 P 2050 5000
 F 0 "D15" V 2004 5079 50  0000 L CNN
-F 1 "BZX84Cxx" V 2095 5079 50  0000 L CNN
+F 1 "BZX84C10LT1G" V 2095 5079 50  0000 L CNN
 F 2 "KiCad/Diode_SMD.pretty:D_SOT-23_ANK" H 2050 4825 50  0001 C CNN
 F 3 "https://diotec.com/tl_files/diotec/files/pdf/datasheets/bzx84c2v4.pdf" H 2050 5000 50  0001 C CNN
@@
 F 3 "https://assets.nexperia.com/documents/data-sheet/BAV99_SER.pdf" H 3650 2250 50  0001 C CNN
 	2    3650 2150
-	-1   0    0    1
+	1    0    0    -1
 $EndComp
 Connection ~ 3500 2150
@@
 F 3 "https://assets.nexperia.com/documents/data-sheet/BAV99_SER.pdf" H 3700 4250 50  0001 C CNN
 	2    3700 4150
-	-1   0    0    1
+	1    0    0    -1
 $EndComp
 Connection ~ 3550 4150

Commit message: mods during bring up, see notes
Parts:
- R65: value 9k1 -> 1k
Changed lines of the file:
@@
 F 1 "3k9" H 2780 5095 50  0000 R CNN
 F 2 "KiCad/Resistor_SMD.pretty:R_0603_1608Metric" V 2780 5050 50  0001 C CNN
-F 3 "~" H 2850 5050 50  0001 C CNN
+F 3 "" H 2850 5050 50  0001 C CNN
 F 4 "0.1%" H 2850 5050 50  0001 C CNN "Characteristics"
 	1    2850 5050
@@
 F 1 "50k" H 3580 9695 50  0000 R CNN
 F 2 "KiCad/Resistor_SMD.pretty:R_0603_1608Metric" V 3580 9650 50  0001 C CNN
-F 3 "~" H 3650 9650 50  0001 C CNN
+F 3 "" H 3650 9650 50  0001 C CNN
 F 4 "0.1%" H 3650 9650 50  0001 C CNN "Characteristics"
 	1    3650 9650
@@
 F 1 "100k" V 4034 9400 50  0000 C CNN
 F 2 "KiCad/Resistor_SMD.pretty:R_0603_1608Metric" V 4080 9400 50  0001 C CNN
-F 3 "~" H 4150 9400 50  0001 C CNN
+F 3 "" H 4150 9400 50  0001 C CNN
 F 4 "0.1%" H 4150 9400 50  0001 C CNN "Characteristics"
 	1    4150 9400
@@
 P 3050 8800
 F 0 "R65" V 2843 8800 50  0000 C CNN
-F 1 "9k1" V 2934 8800 50  0000 C CNN
+F 1 "1k" V 2934 8800 50  0000 C CNN
 F 2 "KiCad/Resistor_SMD.pretty:R_0603_1608Metric" V 2980 8800 50  0001 C CNN
 F 3 "~" H 3050 8800 50  0001 C CNN

Commit message: bring up firmware, all hardware testing and changes rolled into schematic
Parts:
- R13: value 50k -> 100k
Connections:
- net labels added: +5V
Other:
- note added: "0-5 V target output: 0-2.5 V output from DAC; G = 2 ((100 / 100) + 1)"
- note added: "These values will only work using default 3.3 V internal reference"
- note added: "These values will only work using default 3.3 V internal reference for ADC"
- note removed: "0-10 V output to 0-3.3 V for uC DAC. G = 3 ((100 / 50) + 1)"
Changed lines of the file:
@@
-$EndComp
-$Comp
-L power:VCC #PWR06
-U 1 1 5D0A0214
-P 4600 7350
-F 0 "#PWR06" H 4600 7200 50  0001 C CNN
-F 1 "VCC" H 4617 7523 50  0000 C CNN
-F 2 "" H 4600 7350 50  0001 C CNN
-F 3 "" H 4600 7350 50  0001 C CNN
-	1    4600 7350
-	1    0    0    -1
 $EndComp
 $Comp
@@
 P 3650 9650
 F 0 "R13" H 3580 9604 50  0000 R CNN
-F 1 "50k" H 3580 9695 50  0000 R CNN
+F 1 "100k" H 3580 9695 50  0000 R CNN
 F 2 "KiCad/Resistor_SMD.pretty:R_0603_1608Metric" V 3580 9650 50  0001 C CNN
 F 3 "" H 3650 9650 50  0001 C CNN
@@
 	4450 9400 4300 9400
 Text Notes 3250 6750 0    50   ~ 0
-0-10 V output to 0-3.3 V for uC DAC. G = 3 ((100 / 50) + 1)
+0-5 V target output: 0-2.5 V output from DAC; G = 2 ((100 / 100) + 1)
 $Comp
 L Diode:BAV99 D17
@@
 Wire Wire Line
 	1400 2700 2000 2700
+$Comp
+L power:+5V #PWR?
+U 1 1 5D0C1E91
+P 4600 7350
+F 0 "#PWR?" H 4600 7200 50  0001 C CNN
+F 1 "+5V" H 4615 7523 50  0000 C CNN
+F 2 "" H 4600 7350 50  0001 C CNN
+F 3 "" H 4600 7350 50  0001 C CNN
+	1    4600 7350
+	1    0    0    -1
+$EndComp
+Text Notes 2000 1650 0    50   Italic 0
+These values will only work using default 3.3 V internal reference for ADC
+Text Notes 3350 6900 0    50   Italic 0
+These values will only work using default 3.3 V internal reference
 $EndSCHEMATC
