File: whitterm-hat/power.sch (KiCad schematic (older format))
At the start: 21 parts, among them Q1 IRLML6402PBF, Q2 IRLML6402PBF, Q9 IRLML6402PBF, U9 MCP1703A-3302_SOT23

Commit message: pcb sent for production
Parts:
- added D23: KP-2012MGC, KiCad/LED_SMD.pretty:LED_0603_1608Metric, symbol Device:LED
- added R58: 220R, KiCad/Resistor_SMD.pretty:R_0603_1608Metric, symbol Device:R_Small
- TP25, TP26, TP27: footprint KiCad/TestPoint.pretty:TestPoint_Pad_D2.0mm -> KiCad/TestPoint.pretty:TestPoint_Pad_D1.5mm
- renumbered D23 to D13, D13 to D22, R30 to R20, R31 to R30, R32 to R31, R58 to R32, U9 to U7
Connections:
- wire segments 67 -> 70
Changed lines of the file:
@@
 EESchema Schematic File Version 4
 LIBS:whitterm-hat-cache
-EELAYER 26 0
+EELAYER 29 0
 EELAYER END
 $Descr A3 16535 11693
@@
 $EndDescr
 $Comp
-L Regulator_Linear:MCP1703A-3302_SOT23 U9
+L Regulator_Linear:MCP1703A-3302_SOT23 U7
 U 1 1 5AB155FD
 P 7450 4050
-F 0 "U9" H 7300 4175 50  0000 C CNN
+F 0 "U7" H 7300 4175 50  0000 C CNN
 F 1 "MCP1703A-3302_SOT23" H 7450 4175 50  0000 L CNN
 F 2 "KiCad/Package_TO_SOT_SMD.pretty:SOT-23" H 7450 4250 50  0001 C CNN
@@
 $EndComp
 $Comp
-L Device:LED D13
+L Device:LED D22
 U 1 1 5AB185A2
 P 11950 3650
-F 0 "D13" H 11950 3750 50  0000 C CNN
+F 0 "D22" H 11950 3750 50  0000 C CNN
 F 1 "KP-2012MGC" H 11950 3550 50  0000 C CNN
 F 2 "KiCad/LED_SMD.pretty:LED_0603_1608Metric" H 11950 3650 50  0001 C CNN
@@
 $EndComp
 $Comp
-L Device:R_Small R30
+L Device:R_Small R20
 U 1 1 5AB24B72
 P 5600 4550
-F 0 "R30" H 5630 4570 50  0000 L CNN
+F 0 "R20" H 5630 4570 50  0000 L CNN
 F 1 "10k" H 5630 4510 50  0000 L CNN
 F 2 "KiCad/Resistor_SMD.pretty:R_0603_1608Metric" H 5600 4550 50  0001 C CNN
@@
 	7350 7250 7650 7250
 $Comp
-L Device:R_Small R31
+L Device:R_Small R30
 U 1 1 5C672C21
 P 6700 6950
-F 0 "R31" H 6730 6970 50  0000 L CNN
+F 0 "R30" H 6730 6970 50  0000 L CNN
 F 1 "10k" H 6730 6910 50  0000 L CNN
 F 2 "KiCad/Resistor_SMD.pretty:R_0603_1608Metric" H 6700 6950 50  0001 C CNN
@@
 Connection ~ 7350 7250
 $Comp
-L Device:R_Small R32
+L Device:R_Small R31
 U 1 1 5C674B9F
 P 7750 7250
-F 0 "R32" H 7780 7270 50  0000 L CNN
+F 0 "R31" H 7780 7270 50  0000 L CNN
 F 1 "150R" H 7780 7210 50  0000 L CNN
 F 2 "KiCad/Resistor_SMD.pretty:R_0603_1608Metric" H 7750 7250 50  0001 C CNN
@@
 $EndComp
 $Comp
-L Device:R_Small R58
+L Device:R_Small R32
 U 1 1 5D3E3444
 P 10800 7100
-F 0 "R58" H 10830 7120 50  0000 L CNN
+F 0 "R32" H 10830 7120 50  0000 L CNN
 F 1 "10k" H 10830 7060 50  0000 L CNN
 F 2 "KiCad/Resistor_SMD.pretty:R_0603_1608Metric" H 10800 7100 50  0001 C CNN
@@
 	10800 7200 10800 7300
 $Comp
-L Device:D_Zener_Small D23
+L Device:D_Zener_Small D13
 U 1 1 5D3E3455
 P 11250 6800
-F 0 "D23" H 11250 6890 50  0000 C CNN
+F 0 "D13" H 11250 6890 50  0000 C CNN
 F 1 "MMSZ16T1G" V 11500 6800 50  0000 C CNN
 F 2 "KiCad/Diode_SMD.pretty:D_SOD-123" V 11250 6800 50  0001 C CNN
@@
 F 0 "TP27" H 8608 4124 50  0000 L CNN
 F 1 "TestPoint" H 8608 4079 50  0001 L CNN
-F 2 "KiCad/TestPoint.pretty:TestPoint_Pad_D2.0mm" H 8750 4050 50  0001 C CNN
+F 2 "KiCad/TestPoint.pretty:TestPoint_Pad_D1.5mm" H 8750 4050 50  0001 C CNN
 F 3 "~" H 8750 4050 50  0001 C CNN
 	1    8550 4050
@@
 F 0 "TP25" H 5258 4124 50  0000 L CNN
 F 1 "TestPoint" H 5258 4079 50  0001 L CNN
-F 2 "KiCad/TestPoint.pretty:TestPoint_Pad_D2.0mm" H 5400 4050 50  0001 C CNN
+F 2 "KiCad/TestPoint.pretty:TestPoint_Pad_D1.5mm" H 5400 4050 50  0001 C CNN
 F 3 "~" H 5400 4050 50  0001 C CNN
 	1    5200 4050
@@
 F 0 "TP26" H 6658 4124 50  0000 L CNN
 F 1 "TestPoint" H 6658 4079 50  0001 L CNN
-F 2 "KiCad/TestPoint.pretty:TestPoint_Pad_D2.0mm" H 6800 4050 50  0001 C CNN
+F 2 "KiCad/TestPoint.pretty:TestPoint_Pad_D1.5mm" H 6800 4050 50  0001 C CNN
 F 3 "~" H 6800 4050 50  0001 C CNN
 	1    6600 4050
@@
 Wire Wire Line
 	6600 4050 7150 4050
+$Comp
+L Device:LED D23
+U 1 1 5CA2321A
+P 5600 6550
+F 0 "D23" H 5600 6650 50  0000 C CNN
+F 1 "KP-2012MGC" H 5600 6450 50  0000 C CNN
+F 2 "KiCad/LED_SMD.pretty:LED_0603_1608Metric" H 5600 6550 50  0001 C CNN
+F 3 "" H 5600 6550 50  0001 C CNN
+F 4 "Kingbright" H 5600 6550 60  0001 C CNN "MFN"
+F 5 "KP-2012MGC" H 5600 6550 60  0001 C CNN "MFP"
+F 6 "KP-2012MGC Green LED, 570 nm 2012 (0805), Rectangle Lens SMD package" H 5600 6550 60  0001 C CNN "Description"
+	1    5600 6550
+	0    -1   -1   0
+$EndComp
+$Comp
+L Device:R_Small R58
+U 1 1 5CA23226
+P 5600 6900
+F 0 "R58" H 5630 6920 50  0000 L CNN
+F 1 "220R" H 5630 6860 50  0000 L CNN
+F 2 "KiCad/Resistor_SMD.pretty:R_0603_1608Metric" H 5600 6900 50  0001 C CNN
+F 3 "" H 5600 6900 50  0001 C CNN
+	1    5600 6900
+	1    0    0    -1
+$EndComp
+Wire Wire Line
+	5600 6300 5600 6400
+Wire Wire Line
+	5600 6700 5600 6800
+$Comp
+L power:GND #PWR018
+U 1 1 5CA2322E
+P 5600 7100
+F 0 "#PWR018" H 5600 6850 50  0001 C CNN
+F 1 "GND" H 5600 6950 50  0000 C CNN
+F 2 "" H 5600 7100 50  0001 C CNN
+F 3 "" H 5600 7100 50  0001 C CNN
+	1    5600 7100
+	1    0    0    -1
+$EndComp
+Wire Wire Line
+	5600 7000 5600 7100
+Text HLabel 5600 6300 1    50   UnSpc ~ 0
+PI_5V
 $EndSCHEMATC

Commit message: mods during bring up, see notes
Parts:
- removed R31: 150R, KiCad/Resistor_SMD.pretty:R_0603_1608Metric, symbol Device:R_Small
- added Q?: BC850, KiCad/Package_TO_SOT_SMD.pretty:SOT-23, symbol Transistor_BJT:BC850
Connections:
- net labels added: PI_EN
- net labels removed: ~PI_EN
- wire segments 70 -> 72
Changed lines of the file:
@@
 Text HLabel 8100 6650 2    50   UnSpc ~ 0
 PI_5V
-Text HLabel 8100 7250 2    50   Input ~ 0
-~PI_EN
+Text HLabel 8450 7550 2    50   Input ~ 0
+PI_EN
 Wire Wire Line
 	6700 6650 7150 6650
 Wire Wire Line
 	7550 6650 7900 6650
-Wire Wire Line
-	7350 6950 7350 7250
-Wire Wire Line
-	7350 7250 7650 7250
 $Comp
 L Device:R_Small R30
@@
 	6700 7050 6700 7250
 Wire Wire Line
-	6700 7250 7350 7250
-Connection ~ 7350 7250
-$Comp
-L Device:R_Small R31
-U 1 1 5C674B9F
-P 7750 7250
-F 0 "R31" H 7780 7270 50  0000 L CNN
-F 1 "150R" H 7780 7210 50  0000 L CNN
-F 2 "KiCad/Resistor_SMD.pretty:R_0603_1608Metric" H 7750 7250 50  0001 C CNN
-F 3 "" H 7750 7250 50  0001 C CNN
-	1    7750 7250
-	0    1    1    0
-$EndComp
-Wire Wire Line
-	7850 7250 8100 7250
+	8200 7550 8450 7550
 $Comp
 L Device:Jumper_NO_Small JP?
@@
 Text HLabel 5600 6300 1    50   UnSpc ~ 0
 PI_5V
+$Comp
+L power:GND #PWR?
+U 1 1 5D00BC51
+P 7900 7850
+F 0 "#PWR?" H 7900 7600 50  0001 C CNN
+F 1 "GND" H 7900 7700 50  0000 C CNN
+F 2 "" H 7900 7850 50  0001 C CNN
+F 3 "" H 7900 7850 50  0001 C CNN
+	1    7900 7850
+	1    0    0    -1
+$EndComp
+Wire Wire Line
+	7900 7750 7900 7850
+$Comp
+L Transistor_BJT:BC850 Q?
+U 1 1 5CFFBA8C
+P 8000 7550
+AR Path="/5C67462C/5CFFBA8C" Ref="Q?"  Part="1"
+AR Path="/5C65C880/5CFFBA8C" Ref="Q?"  Part="1"
+F 0 "Q?" H 8191 7596 50  0000 L CNN
+F 1 "BC850" H 8191 7505 50  0000 L CNN
+F 2 "KiCad/Package_TO_SOT_SMD.pretty:SOT-23" H 8200 7475 50  0001 L CIN
+F 3 "http://www.infineon.com/dgdl/Infineon-BC847SERIES_BC848SERIES_BC849SERIES_BC850SERIES-DS-v01_01-en.pdf?fileId=db3a304314dca389011541d4630a1657" H 8000 7550 50  0001 L CNN
+	1    8000 7550
+	-1   0    0    -1
+$EndComp
+Wire Wire Line
+	6700 7250 7350 7250
+Wire Wire Line
+	7900 7250 7900 7350
+Wire Wire Line
+	7350 6950 7350 7250
+Connection ~ 7350 7250
+Wire Wire Line
+	7350 7250 7900 7250
 $EndSCHEMATC

Commit message: firmware functionally complete for basic button usage
Parts:
- gave numbers to parts that had none: 1
Changed lines of the file:
@@
 PI_5V
 $Comp
-L power:GND #PWR?
+L power:GND #PWR0161
 U 1 1 5D00BC51
 P 7900 7850
-F 0 "#PWR?" H 7900 7600 50  0001 C CNN
+F 0 "#PWR0161" H 7900 7600 50  0001 C CNN
 F 1 "GND" H 7900 7700 50  0000 C CNN
 F 2 "" H 7900 7850 50  0001 C CNN
@@
 P 8000 7550
 AR Path="/5C67462C/5CFFBA8C" Ref="Q?"  Part="1"
-AR Path="/5C65C880/5CFFBA8C" Ref="Q?"  Part="1"
-F 0 "Q?" H 8191 7596 50  0000 L CNN
+AR Path="/5C65C880/5CFFBA8C" Ref="Q12"  Part="1"
+F 0 "Q12" H 8191 7596 50  0000 L CNN
 F 1 "BC850" H 8191 7505 50  0000 L CNN
 F 2 "KiCad/Package_TO_SOT_SMD.pretty:SOT-23" H 8200 7475 50  0001 L CIN
