File: whitterm-hat/whitterm-hat.sch (KiCad schematic (older format))
At the start: 54 parts, among them J1 USB_C_Receptacle, J2 Touch I2C, J3 40HAT, J6 Conn_01x04_Female, J7 Conn_01x04_Female, J8 Conn_01x10_Female, J9 CONN_01X02, U1 TUSB320, U2 CAT24C32, U3 74LVC1G17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

Commit message: pcb sent for production
Parts:
- removed TP8, TP9: TestPoint, KiCad/TestPoint.pretty:TestPoint_Pad_D2.0mm, symbol Connector:TestPoint
- J3: footprint KiCad/Connector_PinHeader_2.54mm.pretty:PinHeader_2x20_P2.54mm_Vertical -> greatscottgadgets/gsg-kicad-lib/gsg-modules.pretty:HEADER-2x20-REVERSE
- R12: MFR Yageo -> (none); MPN RC0402JR-0722RL -> (none); Notes (none) -> DNF; SPN 311-22JRCT-ND -> (none)
- TP1, TP10, TP11, TP12, TP13, TP14, TP15, TP16, TP2, TP3, TP4, TP5, TP6, TP7: footprint KiCad/TestPoint.pretty:TestPoint_Pad_D2.0mm -> KiCad/TestPoint.pretty:TestPoint_Pad_D1.5mm
Connections:
- net labels added: U_CTS, U_RTS
- net labels removed: PI_CE0, PI_CE1, PI_MISO, PI_MOSI, PI_SCLK
- wire segments 247 -> 246
- no-connect marks 35 -> 34

Commit message: button button logic
Connections:
- wire segments 246 -> 234
Changed lines of the file:
@@
 	2050 7800 2250 7800
 Wire Wire Line
-	2250 7800 2250 7750
-Wire Wire Line
-	2050 7500 2250 7500
-Connection ~ 2250 7500
-Wire Wire Line
-	2050 7600 2250 7600
-Connection ~ 2250 7600
-Wire Wire Line
-	2250 7600 2250 7500
-Wire Wire Line
-	2050 7700 2250 7700
-Connection ~ 2250 7700
-Wire Wire Line
-	2250 7700 2250 7600
-Wire Wire Line
 	3100 7700 2850 7700
-Wire Wire Line
-	2550 7700 2550 7750
-Wire Wire Line
-	2550 7750 2250 7750
-Connection ~ 2250 7750
-Wire Wire Line
-	2250 7750 2250 7700
 $Comp
 L power:VBUS #PWR0111
@@
 	1150 10400 1150 10500
 Wire Wire Line
-	1150 10500 1250 10500
-Wire Wire Line
-	1250 10400 1250 10500
-Connection ~ 1250 10500
-Wire Wire Line
-	1250 10500 1350 10500
-Wire Wire Line
-	1350 10400 1350 10500
-Connection ~ 1350 10500
-Wire Wire Line
-	1350 10500 1450 10500
-Wire Wire Line
 	1450 10400 1450 10500
 Connection ~ 1450 10500
 Wire Wire Line
 	1450 10500 1550 10500
-Wire Wire Line
-	1550 10400 1550 10500
-Connection ~ 1550 10500
 $Comp
 L Device:Jumper_NO_Small JP5
@@
 ~PI_EN
 Wire Wire Line
-	2250 7250 2250 7500
-Wire Wire Line
 	3400 7250 3400 8250
 Wire Wire Line
@@
 	0    1    1    0
 $EndComp
+Wire Wire Line
+	2250 7250 2250 7800
+Wire Wire Line
+	2550 7800 2250 7800
+Wire Wire Line
+	2550 7700 2550 7800
+Connection ~ 2250 7800
+Wire Wire Line
+	1150 10500 1450 10500
 $EndSCHEMATC

Commit message: mods during bring up, see notes
Parts:
- added J?: Conn_01x04_Female, KiCad/Connector_PinHeader_2.54mm.pretty:PinHeader_1x04_P2.54mm_Vertical, symbol Connector:Conn_01x04_Female
- added R? (x2): 10k, KiCad/Resistor_SMD.pretty:R_0603_1608Metric, symbol Device:R_Small
- R10, R47, R6, R8: value 3.9K -> 4.7K; MFR Yageo -> (none); MPN RC0402JR-0722RL -> (none); SPN 311-22JRCT-ND -> (none); SPR Digikey -> (none)
- R11, R29: MFR Yageo -> (none); MPN RC0402JR-0722RL -> (none); SPN 311-22JRCT-ND -> (none); SPR Digikey -> (none)
- R12: value 3.9K -> 4.7K; SPR Digikey -> (none)
- R48: value 3.9K -> 4.7K; MFR Yageo -> (none); MPN RC0402JR-0722RL -> (none); SPN 311-22JRCT-ND -> (none)
- R7, R9: value 110R -> 150R
- U2: value CAT24C32 -> CAT24C32WI-GT3; Description (none) -> IC EEPROM 32K I2C 1MHZ 8SOIC; MFN (none) -> ON Semiconductor; MFP (none) -> CAT24C32WI-GT3
Connections:
- net labels added: PI_EN
- net labels removed: ~PI_EN
- wire segments 234 -> 244

Commit message: bring up firmware, all hardware testing and changes rolled into schematic
Changed lines of the file:
@@
 F6 "DOUT_O1" I R 13900 4550 50
 F7 "DOUT_I1" I L 12350 4550 50
-F8 "DIN_O1" I R 13900 4750 50
-F9 "DIN_I1" I L 12350 4750 50
+F8 "DIN_O1" I L 12350 4750 50
+F9 "DIN_I1" I R 13900 4750 50
 F10 "AOUT_I1" I L 12350 5050 50
 F11 "AOUT_O1" I R 13900 5050 50
 F12 "DOUT_O2" I R 13900 4650 50
 F13 "DOUT_I2" I L 12350 4650 50
-F14 "DIN_O2" I R 13900 4850 50
-F15 "DIN_I2" I L 12350 4850 50
+F14 "DIN_O2" I L 12350 4850 50
+F15 "DIN_I2" I R 13900 4850 50
 $EndSheet
 $Comp
@@
 	11350 4650 12350 4650
 Wire Wire Line
-	11350 4750 12350 4750
-Wire Wire Line
-	11350 4850 12350 4850
-Wire Wire Line
 	11350 5050 12350 5050
 $Comp
@@
 Wire Wire Line
 	13900 4650 14900 4650
-Wire Wire Line
-	13900 4750 14900 4750
-Wire Wire Line
-	13900 4850 14900 4850
 Wire Wire Line
 	13900 5050 14050 5050
@@
 Wire Wire Line
 	14650 2600 14900 2600
+Wire Wire Line
+	13900 4850 14900 4850
+Wire Wire Line
+	13900 4750 14900 4750
+Wire Wire Line
+	12350 4750 11350 4750
+Wire Wire Line
+	12350 4850 11350 4850
 $EndSCHEMATC

Commit message: firmware functionally complete for basic button usage
Parts:
- gave numbers to parts that had none: 3
Changed lines of the file:
@@
 	1150 10500 1450 10500
 $Comp
-L Device:R_Small R?
+L Device:R_Small R31
 U 1 1 5CFD4592
 P 5300 7500
-F 0 "R?" V 5400 7500 50  0000 C CNN
+F 0 "R31" V 5400 7500 50  0000 C CNN
 F 1 "10k" V 5400 7350 50  0000 C CNN
 F 2 "KiCad/Resistor_SMD.pretty:R_0603_1608Metric" H 5300 7500 50  0001 C CNN
@@
 $EndComp
 $Comp
-L Device:R_Small R?
+L Device:R_Small R67
 U 1 1 5CFD49F1
 P 5500 7500
-F 0 "R?" V 5600 7500 50  0000 C CNN
+F 0 "R67" V 5600 7500 50  0000 C CNN
 F 1 "10k" V 5600 7350 50  0000 C CNN
 F 2 "KiCad/Resistor_SMD.pretty:R_0603_1608Metric" H 5500 7500 50  0001 C CNN
@@
 $EndComp
 $Comp
-L power:VCC #PWR?
+L power:VCC #PWR0159
 U 1 1 5CFD4F09
 P 5300 7250
-F 0 "#PWR?" H 5300 7100 50  0001 C CNN
+F 0 "#PWR0159" H 5300 7100 50  0001 C CNN
 F 1 "VCC" H 5317 7423 50  0000 C CNN
 F 2 "" H 5300 7250 50  0001 C CNN
@@
 $EndComp
 $Comp
-L power:VCC #PWR?
+L power:VCC #PWR0160
 U 1 1 5CFD5324
 P 5500 7250
-F 0 "#PWR?" H 5500 7100 50  0001 C CNN
+F 0 "#PWR0160" H 5500 7100 50  0001 C CNN
 F 1 "VCC" H 5517 7423 50  0000 C CNN
 F 2 "" H 5500 7250 50  0001 C CNN
@@
 	5500 7900 6550 7900
 $Comp
-L Connector:Conn_01x04_Female J?
+L Connector:Conn_01x04_Female J10
 U 1 1 5D0C3A01
 P 15100 2700
-F 0 "J?" H 15127 2676 50  0000 L CNN
+F 0 "J10" H 15127 2676 50  0000 L CNN
 F 1 "Conn_01x04_Female" H 15127 2585 50  0000 L CNN
 F 2 "KiCad/Connector_PinHeader_2.54mm.pretty:PinHeader_1x04_P2.54mm_Vertical" H 15100 2700 50  0001 C CNN
