File: whitterm-hat/RS232-UART.sch (KiCad schematic (older format))
At the start: 47 parts, among them J4 DB9_Male, Q10 BC850, Q11 BC850, Q7 IRLML6402PBF, Q8 IRLML6402PBF, SW1 SW_DIP_x06, U5 MAX3221, U6 74LVC2G02

Commit message: pcb sent for production
Parts:
- removed R20: 10k, KiCad/Resistor_SMD.pretty:R_0603_1608Metric, symbol Device:R
- D7: value RXD -> TXD
- TP17, TP18, TP19, TP20, TP21, TP34, TP35, TP36, TP37: footprint KiCad/TestPoint.pretty:TestPoint_Pad_D2.0mm -> KiCad/TestPoint.pretty:TestPoint_Pad_D1.5mm
Connections:
- wire segments 154 -> 151
Changed lines of the file:
@@
 EESchema Schematic File Version 4
 LIBS:whitterm-hat-cache
-EELAYER 26 0
+EELAYER 29 0
 EELAYER END
 $Descr A3 16535 11693
@@
 ON ACT LED PCHAN\n0    0         0   1\n1     0         1   0\n0    1          1   0\n1     1         1   0
 $Comp
-L Device:R R20
-U 1 1 5C572E82
-P 11000 7850
-F 0 "R20" V 11100 7850 50  0000 C CNN
-F 1 "10k" V 10900 7850 50  0000 C CNN
-F 2 "KiCad/Resistor_SMD.pretty:R_0603_1608Metric" V 10930 7850 50  0001 C CNN
-F 3 "~" H 11000 7850 50  0001 C CNN
-	1    11000 7850
-	-1   0    0    1
-$EndComp
-$Comp
 L Device:R R21
 U 1 1 5C573548
@@
 P 12200 7400
 F 0 "D7" V 12238 7283 50  0000 R CNN
-F 1 "RXD" V 12147 7283 50  0000 R CNN
+F 1 "TXD" V 12147 7283 50  0000 R CNN
 F 2 "KiCad/LED_SMD.pretty:LED_0603_1608Metric" H 12200 7400 50  0001 C CNN
 F 3 "~" H 12200 7400 50  0001 C CNN
@@
 F 0 "TP17" H 2558 4524 50  0000 L CNN
 F 1 "TestPoint" H 2558 4479 50  0001 L CNN
-F 2 "KiCad/TestPoint.pretty:TestPoint_Pad_D2.0mm" H 2700 4450 50  0001 C CNN
+F 2 "KiCad/TestPoint.pretty:TestPoint_Pad_D1.5mm" H 2700 4450 50  0001 C CNN
 F 3 "~" H 2700 4450 50  0001 C CNN
 	1    2500 4450
@@
 F 0 "TP18" H 2558 4724 50  0000 L CNN
 F 1 "TestPoint" H 2558 4679 50  0001 L CNN
-F 2 "KiCad/TestPoint.pretty:TestPoint_Pad_D2.0mm" H 2700 4650 50  0001 C CNN
+F 2 "KiCad/TestPoint.pretty:TestPoint_Pad_D1.5mm" H 2700 4650 50  0001 C CNN
 F 3 "~" H 2700 4650 50  0001 C CNN
 	1    2500 4650
@@
 F 0 "TP21" H 12658 6324 50  0000 L CNN
 F 1 "TestPoint" H 12658 6279 50  0001 L CNN
-F 2 "KiCad/TestPoint.pretty:TestPoint_Pad_D2.0mm" H 12800 6250 50  0001 C CNN
+F 2 "KiCad/TestPoint.pretty:TestPoint_Pad_D1.5mm" H 12800 6250 50  0001 C CNN
 F 3 "~" H 12800 6250 50  0001 C CNN
 	1    12600 6250
@@
 F 0 "TP19" H 7458 3824 50  0000 L CNN
 F 1 "TestPoint" H 7458 3779 50  0001 L CNN
-F 2 "KiCad/TestPoint.pretty:TestPoint_Pad_D2.0mm" H 7600 3750 50  0001 C CNN
+F 2 "KiCad/TestPoint.pretty:TestPoint_Pad_D1.5mm" H 7600 3750 50  0001 C CNN
 F 3 "~" H 7600 3750 50  0001 C CNN
 	1    7400 3750
@@
 F 0 "TP20" H 7858 3924 50  0000 L CNN
 F 1 "TestPoint" H 7858 3879 50  0001 L CNN
-F 2 "KiCad/TestPoint.pretty:TestPoint_Pad_D2.0mm" H 8000 3850 50  0001 C CNN
+F 2 "KiCad/TestPoint.pretty:TestPoint_Pad_D1.5mm" H 8000 3850 50  0001 C CNN
 F 3 "~" H 8000 3850 50  0001 C CNN
 	1    7800 3850
@@
 Wire Wire Line
 	10800 8100 11250 8100
-$Comp
-L power:VCC #PWR018
-U 1 1 5C85C151
-P 11000 7600
-F 0 "#PWR018" H 11000 7450 50  0001 C CNN
-F 1 "VCC" H 11017 7773 50  0000 C CNN
-F 2 "" H 11000 7600 50  0001 C CNN
-F 3 "" H 11000 7600 50  0001 C CNN
-	1    11000 7600
-	1    0    0    -1
-$EndComp
-Wire Wire Line
-	11000 7600 11000 7700
-Wire Wire Line
-	11000 8000 11000 8200
-Connection ~ 11000 8200
-Wire Wire Line
-	11000 8200 11250 8200
-Wire Wire Line
-	10800 8200 11000 8200
 Wire Wire Line
 	10950 5700 10950 5800
@@
 F 0 "TP34" H 12658 8224 50  0000 L CNN
 F 1 "TestPoint" H 12658 8179 50  0001 L CNN
-F 2 "KiCad/TestPoint.pretty:TestPoint_Pad_D2.0mm" H 12800 8150 50  0001 C CNN
+F 2 "KiCad/TestPoint.pretty:TestPoint_Pad_D1.5mm" H 12800 8150 50  0001 C CNN
 F 3 "~" H 12800 8150 50  0001 C CNN
 	1    12600 8150
@@
 F 0 "TP35" H 5758 5924 50  0000 L CNN
 F 1 "TestPoint" H 5758 5879 50  0001 L CNN
-F 2 "KiCad/TestPoint.pretty:TestPoint_Pad_D2.0mm" H 5900 5850 50  0001 C CNN
+F 2 "KiCad/TestPoint.pretty:TestPoint_Pad_D1.5mm" H 5900 5850 50  0001 C CNN
 F 3 "~" H 5900 5850 50  0001 C CNN
 	1    5700 5850
@@
 F 0 "TP36" H 5808 9174 50  0000 L CNN
 F 1 "TestPoint" H 5808 9129 50  0001 L CNN
-F 2 "KiCad/TestPoint.pretty:TestPoint_Pad_D2.0mm" H 5950 9100 50  0001 C CNN
+F 2 "KiCad/TestPoint.pretty:TestPoint_Pad_D1.5mm" H 5950 9100 50  0001 C CNN
 F 3 "~" H 5950 9100 50  0001 C CNN
 	1    5750 9100
@@
 F 0 "TP37" H 6708 6524 50  0000 L CNN
 F 1 "TestPoint" H 6708 6479 50  0001 L CNN
-F 2 "KiCad/TestPoint.pretty:TestPoint_Pad_D2.0mm" H 6850 6450 50  0001 C CNN
+F 2 "KiCad/TestPoint.pretty:TestPoint_Pad_D1.5mm" H 6850 6450 50  0001 C CNN
 F 3 "~" H 6850 6450 50  0001 C CNN
 	1    6650 6450
@@
 Wire Wire Line
 	6650 6450 6950 6450
+Wire Wire Line
+	10800 8200 11250 8200
 $EndSCHEMATC

Commit message: mods during bring up, see notes
Parts:
- R18, R19, R22, R23: value 110R -> 150R
Changed lines of the file:
@@
 P 7600 3350
 F 0 "R18" V 7393 3350 50  0000 C CNN
-F 1 "110R" V 7484 3350 50  0000 C CNN
+F 1 "150R" V 7484 3350 50  0000 C CNN
 F 2 "KiCad/Resistor_SMD.pretty:R_0603_1608Metric" V 7530 3350 50  0001 C CNN
 F 3 "~" H 7600 3350 50  0001 C CNN
@@
 P 8000 3350
 F 0 "R19" V 7793 3350 50  0000 C CNN
-F 1 "110R" V 7884 3350 50  0000 C CNN
+F 1 "150R" V 7884 3350 50  0000 C CNN
 F 2 "KiCad/Resistor_SMD.pretty:R_0603_1608Metric" V 7930 3350 50  0001 C CNN
 F 3 "~" H 8000 3350 50  0001 C CNN
@@
 P 12200 5950
 F 0 "R22" V 11993 5950 50  0000 C CNN
-F 1 "110R" V 12084 5950 50  0000 C CNN
+F 1 "150R" V 12084 5950 50  0000 C CNN
 F 2 "KiCad/Resistor_SMD.pretty:R_0603_1608Metric" V 12130 5950 50  0001 C CNN
 F 3 "~" H 12200 5950 50  0001 C CNN
@@
 P 12200 7800
 F 0 "R23" V 11993 7800 50  0000 C CNN
-F 1 "110R" V 12084 7800 50  0000 C CNN
+F 1 "150R" V 12084 7800 50  0000 C CNN
 F 2 "KiCad/Resistor_SMD.pretty:R_0603_1608Metric" V 12130 7800 50  0001 C CNN
 F 3 "~" H 12200 7800 50  0001 C CNN

Commit message: buffer on RS232 LEDs
Parts:
- added U? (x2): 74LVC1G17, KiCad/Package_TO_SOT_SMD.pretty:TSOT-23-5, symbol 74xGxx:74LVC1G17
- U5: footprint KiCad/Package_SO.pretty:TSSOP-16_4.4x5mm_P0.65mm -> fruchti/fruchtilib/mod/tssop.pretty:TSSOP16
Connections:
- wire segments 151 -> 153
Changed lines of the file:
@@
 F 0 "U5" H 6150 4428 50  0000 C CNN
 F 1 "MAX3221" H 6150 4337 50  0000 C CNN
-F 2 "KiCad/Package_SO.pretty:TSSOP-16_4.4x5mm_P0.65mm" H 6200 3350 50  0001 C CIN
+F 2 "fruchti/fruchtilib/mod/tssop.pretty:TSSOP16" H 6200 3350 50  0001 C CIN
 F 3 "http://www.ti.com/lit/ds/symlink/max3221.pdf" H 6150 4300 50  0001 C CNN
 	1    6150 3350
@@
 L Device:LED D4
 U 1 1 5C55BD50
-P 7600 2850
-F 0 "D4" V 7638 2733 50  0000 R CNN
-F 1 "TLRX" V 7547 2733 50  0000 R CNN
-F 2 "KiCad/LED_SMD.pretty:LED_0603_1608Metric" H 7600 2850 50  0001 C CNN
-F 3 "~" H 7600 2850 50  0001 C CNN
-F 4 "Kingbright" H 7600 2850 50  0001 C CNN "MFN"
-F 5 "KP-2012SEC" H 7600 2850 50  0001 C CNN "MFP"
-F 6 "Orange" H 7600 2850 50  0001 C CNN "Characteristics"
-F 7 "RS232 LED" H 7600 2850 50  0001 C CNN "Description"
-	1    7600 2850
+P 7600 2200
+F 0 "D4" V 7638 2083 50  0000 R CNN
+F 1 "TLRX" V 7547 2083 50  0000 R CNN
+F 2 "KiCad/LED_SMD.pretty:LED_0603_1608Metric" H 7600 2200 50  0001 C CNN
+F 3 "~" H 7600 2200 50  0001 C CNN
+F 4 "Kingbright" H 7600 2200 50  0001 C CNN "MFN"
+F 5 "KP-2012SEC" H 7600 2200 50  0001 C CNN "MFP"
+F 6 "Orange" H 7600 2200 50  0001 C CNN "Characteristics"
+F 7 "RS232 LED" H 7600 2200 50  0001 C CNN "Description"
+	1    7600 2200
 	0    -1   -1   0
 $EndComp
@@
 L Device:LED D5
 U 1 1 5C55C45D
-P 8000 2850
-F 0 "D5" V 8038 2733 50  0000 R CNN
-F 1 "TLTX" V 7947 2733 50  0000 R CNN
-F 2 "KiCad/LED_SMD.pretty:LED_0603_1608Metric" H 8000 2850 50  0001 C CNN
-F 3 "~" H 8000 2850 50  0001 C CNN
-F 4 "Kingbright" H 8000 2850 50  0001 C CNN "MFN"
-F 5 "KP-2012SEC" H 8000 2850 50  0001 C CNN "MFP"
-F 6 "Orange" H 8000 2850 50  0001 C CNN "Characteristics"
-F 7 "RS232 LED" H 8000 2850 50  0001 C CNN "Description"
-	1    8000 2850
+P 8000 2200
+F 0 "D5" V 8038 2083 50  0000 R CNN
+F 1 "TLTX" V 7947 2083 50  0000 R CNN
+F 2 "KiCad/LED_SMD.pretty:LED_0603_1608Metric" H 8000 2200 50  0001 C CNN
+F 3 "~" H 8000 2200 50  0001 C CNN
+F 4 "Kingbright" H 8000 2200 50  0001 C CNN "MFN"
+F 5 "KP-2012SEC" H 8000 2200 50  0001 C CNN "MFP"
+F 6 "Orange" H 8000 2200 50  0001 C CNN "Characteristics"
+F 7 "RS232 LED" H 8000 2200 50  0001 C CNN "Description"
+	1    8000 2200
 	0    -1   -1   0
 $EndComp
@@
 L Device:R R18
 U 1 1 5C55DDB6
-P 7600 3350
-F 0 "R18" V 7393 3350 50  0000 C CNN
-F 1 "150R" V 7484 3350 50  0000 C CNN
-F 2 "KiCad/Resistor_SMD.pretty:R_0603_1608Metric" V 7530 3350 50  0001 C CNN
-F 3 "~" H 7600 3350 50  0001 C CNN
-	1    7600 3350
+P 7600 2700
+F 0 "R18" V 7393 2700 50  0000 C CNN
+F 1 "150R" V 7484 2700 50  0000 C CNN
+F 2 "KiCad/Resistor_SMD.pretty:R_0603_1608Metric" V 7530 2700 50  0001 C CNN
+F 3 "~" H 7600 2700 50  0001 C CNN
+	1    7600 2700
 	-1   0    0    1
 $EndComp
@@
 L Device:R R19
 U 1 1 5C55E03F
-P 8000 3350
-F 0 "R19" V 7793 3350 50  0000 C CNN
-F 1 "150R" V 7884 3350 50  0000 C CNN
-F 2 "KiCad/Resistor_SMD.pretty:R_0603_1608Metric" V 7930 3350 50  0001 C CNN
-F 3 "~" H 8000 3350 50  0001 C CNN
-	1    8000 3350
+P 8000 2700
+F 0 "R19" V 7793 2700 50  0000 C CNN
+F 1 "150R" V 7884 2700 50  0000 C CNN
+F 2 "KiCad/Resistor_SMD.pretty:R_0603_1608Metric" V 7930 2700 50  0001 C CNN
+F 3 "~" H 8000 2700 50  0001 C CNN
+	1    8000 2700
 	-1   0    0    1
 $EndComp
@@
 L power:VCC #PWR0104
 U 1 1 5C55E968
-P 7600 2400
-F 0 "#PWR0104" H 7600 2250 50  0001 C CNN
-F 1 "VCC" H 7617 2573 50  0000 C CNN
-F 2 "" H 7600 2400 50  0001 C CNN
-F 3 "" H 7600 2400 50  0001 C CNN
-	1    7600 2400
-	1    0    0    -1
-$EndComp
-Wire Wire Line
-	7600 2600 8000 2600
-Wire Wire Line
-	8000 2600 8000 2700
-Connection ~ 7600 2600
-Wire Wire Line
-	7600 2600 7600 2700
-Wire Wire Line
-	7600 2400 7600 2600
-Wire Wire Line
-	7600 3000 7600 3200
-Wire Wire Line
-	8000 3000 8000 3200
-Connection ~ 7600 3750
-Wire Wire Line
-	7600 3750 8250 3750
-Wire Wire Line
-	8000 3500 8000 3850
-Connection ~ 8000 3850
-Wire Wire Line
-	8000 3850 8250 3850
-Wire Wire Line
-	7600 3500 7600 3750
+P 7600 1750
+F 0 "#PWR0104" H 7600 1600 50  0001 C CNN
+F 1 "VCC" H 7617 1923 50  0000 C CNN
+F 2 "" H 7600 1750 50  0001 C CNN
+F 3 "" H 7600 1750 50  0001 C CNN
+	1    7600 1750
+	1    0    0    -1
+$EndComp
+Wire Wire Line
+	7600 1950 8000 1950
+Wire Wire Line
+	8000 1950 8000 2050
+Connection ~ 7600 1950
+Wire Wire Line
+	7600 1950 7600 2050
+Wire Wire Line
+	7600 1750 7600 1950
+Wire Wire Line
+	7600 2350 7600 2550
+Wire Wire Line
+	8000 2350 8000 2550
 Text Notes 12650 5200 0    50   ~ 0
 ON ACT LED PCHAN\n0    0         0   1\n1     0         1   0\n0    1          1   0\n1     1         1   0
@@
 $EndComp
 Connection ~ 7400 3750
-Wire Wire Line
-	7400 3750 7600 3750
 $Comp
 L Connector:TestPoint TP?
@@
 $EndComp
 Connection ~ 7800 3850
-Wire Wire Line
-	7800 3850 8000 3850
 $Comp
 L 74xGxx:74LVC2G02 U6
@@
 Wire Wire Line
 	10800 8200 11250 8200
+$Comp
+L 74xGxx:74LVC1G17 U?
+U 1 1 5D1A27F5
+P 7600 3250
+AR Path="/5C556852/5D1A27F5" Ref="U?"  Part="1"
+AR Path="/5D1A27F5" Ref="U?"  Part="1"
+F 0 "U?" H 7575 3517 50  0000 C CNN
+F 1 "74LVC1G17" H 7575 3426 50  0000 C CNN
+F 2 "KiCad/Package_TO_SOT_SMD.pretty:TSOT-23-5" H 7600 3250 50  0001 C CNN
+F 3 "http://www.ti.com/lit/sg/scyt129e/scyt129e.pdf" H 7600 3250 50  0001 C CNN
+F 4 "Texas Instruments" H 7600 3250 50  0001 C CNN "MFN"
+F 5 "SN74LVC1G17DBVT" H 7600 3250 50  0001 C CNN "MFP"
+	1    7600 3250
+	0    -1   -1   0
+$EndComp
+$Comp
+L 74xGxx:74LVC1G17 U?
+U 1 1 5D1A27FD
+P 8000 3250
+AR Path="/5C556852/5D1A27FD" Ref="U?"  Part="1"
+AR Path="/5D1A27FD" Ref="U?"  Part="1"
+F 0 "U?" H 7975 3517 50  0000 C CNN
+F 1 "74LVC1G17" H 7975 3426 50  0000 C CNN
+F 2 "KiCad/Package_TO_SOT_SMD.pretty:TSOT-23-5" H 8000 3250 50  0001 C CNN
+F 3 "http://www.ti.com/lit/sg/scyt129e/scyt129e.pdf" H 8000 3250 50  0001 C CNN
+F 4 "Texas Instruments" H 8000 3250 50  0001 C CNN "MFN"
+F 5 "SN74LVC1G17DBVT" H 8000 3250 50  0001 C CNN "MFP"
+	1    8000 3250
+	0    -1   -1   0
+$EndComp
+Wire Wire Line
+	7400 3750 7600 3750
+Wire Wire Line
+	7800 3850 8000 3850
+Wire Wire Line
+	7600 2850 7600 3000
+Wire Wire Line
+	8000 2850 8000 3000
+Wire Wire Line
+	7600 3550 7600 3750
+Connection ~ 7600 3750
+Wire Wire Line
+	7600 3750 8250 3750
+Wire Wire Line
+	8000 3550 8000 3850
+Connection ~ 8000 3850
+Wire Wire Line
+	8000 3850 8250 3850
 $EndSCHEMATC
